File: sensor_bar_unified_muxing_1/sensor_bar_unified_muxing_1.kicad_sch (KiCad schematic)
At the start: 86 parts, among them J1 TSW-120-20-S-D-LL, U1 Teensy4.1, U10 DRV5055A1xLPGxQ1, U11 DRV5055A1xLPGxQ1, U12 DRV5055A1xLPGxQ1, U13 DRV5055A1xLPGxQ1, U14 DRV5055A1xLPGxQ1, U15 DRV5055A1xLPGxQ1, U16 DRV5055A1xLPGxQ1, U17 DRV5055A1xLPGxQ1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

Commit message: cleanup
Connections:
- net at JP23.2 (B): now also U1.48 (VIN); no longer U1.49 (VUSB)
Other:
- moved on the sheet: U1

Commit message: design PCB
Signed-off-by: Sawyer Bergeron <sawyerbergeron@gmail.com>
Parts:
- U2, U3: footprint Package_TO_SOT_THT:TO-92_Inline -> Package_TO_SOT_THT:TO-92_Inline_Wide
- U4, U5: footprint Package_TO_SOT_THT:TO-92_Inline -> Package_TO_SOT_THT:TO-92_Wide
Connections:
- net at J1.04, JP9.1 (A), JPE02.1 (A): now also U1.17 (25_A11_RX6_SDA2); no longer U1.32 (40_A16)
- net at J1.12, JP13.1 (A), JPE06.1 (A): now also U1.32 (40_A16); no longer U1.18 (26_A12_MOSI1)
- net at J1.10, JP12.1 (A), JPE05.1 (A): now also U1.33 (41_A17); no longer U1.19 (27_A13_SCK1)
- net at J1.08, JP11.1 (A), JPE04.1 (A): now also U1.19 (27_A13_SCK1); no longer U1.30 (38_CS1_IN1)
- net at J1.06, JP10.1 (A), JPE03.1 (A): now also U1.18 (26_A12_MOSI1); no longer U1.31 (39_MISO1_OUT1A)
- net at J1.14, JP14.1 (A), JPE07.1 (A): now also U1.31 (39_MISO1_OUT1A); no longer U1.17 (25_A11_RX6_SDA2)
- net at J1.02, JP8.1 (A), JPE01.1 (A): now also U1.16 (24_A10_TX6_SCL2); no longer U1.33 (41_A17)
- net at J1.16, JP15.1 (A), JPE08.1 (A): now also U1.30 (38_CS1_IN1); no longer U1.16 (24_A10_TX6_SCL2)
- net at BOARDSEL_CMP1.12 (4A), J1.07: now also U1.5 (3_LRCLK2); no longer U1.2 (0_RX1_CRX2_CS1)
- net at BOARDSEL_CMP1.8 (3A), J1.05: now also U1.4 (2_OUT2); no longer U1.3 (1_TX1_CTX2_MISO1)
- net at BOARDSEL_CMP1.5 (2A), J1.03: now also U1.3 (1_TX1_CTX2_MISO1); no longer U1.4 (2_OUT2)
- net at BOARDSEL_CMP1.1 (1A), J1.01: now also U1.2 (0_RX1_CRX2_CS1); no longer U1.5 (3_LRCLK2)
Other:
- moved on the sheet: BOARDSEL_CMP1, BOARDSEL_ENABLE1, J1, JP1, JP2, JP3, JP4, U1
