File: sensor_bar_unified_muxing_1/sensor_bar_unified_muxing_1.kicad_pcb (KiCad board)
At the start: 2 copper layers, 266 x 63 mm, 110 parts, among them J1 TSW-120-20-S-D-LL, U1 Teensy4.1, U10 DRV5055A1xLPGxQ1, U11 DRV5055A1xLPGxQ1, U12 DRV5055A1xLPGxQ1, U13 DRV5055A1xLPGxQ1, U14 DRV5055A1xLPGxQ1, U15 DRV5055A1xLPGxQ1, U16 DRV5055A1xLPGxQ1, U17 DRV5055A1xLPGxQ1, U18 DRV5055A1xLPGxQ1, U19 DRV5055A1xLPGxQ1, U2 DRV5055A1xLPGxQ1, U3 DRV5055A1xLPGxQ1, U4 DRV5055A1xLPGxQ1, U5 DRV5055A1xLPGxQ1, U6 DRV5055A1xLPGxQ1, U7 DRV5055A1xLPGxQ1, U8 DRV5055A1xLPGxQ1, U9 DRV5055A1xLPGxQ1

Commit message: design PCB
Signed-off-by: Sawyer Bergeron <sawyerbergeron@gmail.com>
Parts:
- removed JP24, JP25, JP26, JP27, JP28, JP29, JP30, JP31, JP32, JP33, JP34, JP35, JP36, JP37, JP38, JP39, JP40, JP41, JP42, JP43, JP44, JP5, JP6, JP7: SolderJumper_2_Open, Jumper:SolderJumper-2_P1.3mm_Open_TrianglePad1.0x1.5mm
- JP10, JP11, JP12, JP13, JP14, JP15, JP16, JP17, JP18, JP19, JP20, JP21, JP22, JP45, JP46, JP47, JP8, JP9, JPE01, JPE02, JPE03, JPE04, JPE05, JPE06, JPE07, JPE08, JPE09, JPE10, JPE11, JPE12, JPE13, JPE14, JPE15, JPE16, JPE17, JPE18: moved to B.Cu
- U10, U11, U12, U13, U14, U15, U16, U17, U18, U19, U2, U3, U4, U5, U6, U7, U8, U9: footprint Package_TO_SOT_THT:TO-92_Inline -> Package_TO_SOT_THT:TO-92_Inline_Wide
- moved JPE01 232.9 mm to (23.2, 55.5), turned to -90 degrees
- moved JPE02 231.0 mm to (25.8, 55.5), turned to -90 degrees
- moved JPE03 229.0 mm to (28.2, 55.5), turned to -90 degrees
- moved JPE04 227.1 mm to (30.8, 55.5), turned to -90 degrees
- moved JPE05 225.0 mm to (33.5, 55.5), turned to -90 degrees
- moved JPE06 223.2 mm to (36.0, 55.5), turned to -90 degrees
- moved JPE07 221.3 mm to (38.5, 55.5), turned to -90 degrees
- moved JPE08 219.5 mm to (41.0, 55.5), turned to -90 degrees
- moved JPE09 217.7 mm to (43.5, 55.5), turned to -90 degrees
- moved JPE10 215.9 mm to (46.0, 55.5), turned to -90 degrees
- moved JPE11 214.2 mm to (48.5, 55.5), turned to -90 degrees
- moved JPE12 212.5 mm to (51.0, 55.5), turned to -90 degrees
- moved JPE13 210.8 mm to (53.5, 55.5), turned to -90 degrees
- moved JPE14 209.1 mm to (56.0, 55.5), turned to -90 degrees
- moved JPE15 207.4 mm to (58.5, 55.5), turned to -90 degrees
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Connections:
- U1 pad 16: Net-(JP15-A) -> Net-(JP8-A)
- U1 pad 17: Net-(JP14-A) -> Net-(JP9-A)
- U1 pad 18: Net-(JP13-A) -> Net-(JP10-A)
- U1 pad 19: Net-(JP12-A) -> Net-(JP11-A)
- U1 pad 2: Net-(BOARDSEL_CMP1-4A) -> Net-(BOARDSEL_CMP1-1A)
- U1 pad 3: Net-(BOARDSEL_CMP1-3A) -> Net-(BOARDSEL_CMP1-2A)
- U1 pad 30: Net-(JP11-A) -> Net-(JP15-A)
- U1 pad 31: Net-(JP10-A) -> Net-(JP14-A)
- U1 pad 32: Net-(JP9-A) -> Net-(JP13-A)
- U1 pad 33: Net-(JP8-A) -> Net-(JP12-A)
- U1 pad 4: Net-(BOARDSEL_CMP1-2A) -> Net-(BOARDSEL_CMP1-3A)
- U1 pad 48: unconnected-(U1-VIN-Pad48) -> Net-(JP23-B)
- U1 pad 49: Net-(JP23-B) -> unconnected-(U1-VUSB-Pad49)
- U1 pad 5: Net-(BOARDSEL_CMP1-1A) -> Net-(BOARDSEL_CMP1-4A)
Routing:
- net GND: track 0.00 -> 706.3 mm, vias 0 -> 10
- net Net-(BOARDSEL_CMP1-VCC): track 0.00 -> 677.8 mm, vias 0 -> 10
- net Net-(JP65-A): track 0.00 -> 270.3 mm, vias 0 -> 1
- net Net-(JP64-A): track 0.00 -> 257.6 mm, vias 0 -> 1
- net Net-(JP10-B): track 0.00 -> 245.1 mm, vias 0 -> 1
- net Net-(JP11-B): track 0.00 -> 232.4 mm, vias 0 -> 1
- net Net-(JP12-B): track 0.00 -> 219.9 mm, vias 0 -> 1
- net Net-(JP13-B): track 0.00 -> 207.3 mm, vias 0 -> 1
- net Net-(BOARDSEL_CMP1-4A): track 0.00 -> 203.2 mm
- net Net-(BOARDSEL_CMP1-2A): track 0.00 -> 200.1 mm
- net Net-(JP14-B): track 0.00 -> 195.0 mm, vias 0 -> 1
- net Net-(BOARDSEL_CMP1-3A): track 0.00 -> 193.2 mm
- net Net-(BOARDSEL_CMP1-1A): track 0.00 -> 186.6 mm
- net Net-(JP15-B): track 0.00 -> 182.1 mm, vias 0 -> 1
- net Net-(JP16-B): track 0.00 -> 169.5 mm, vias 0 -> 1
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Other:
- board size 266 x 63 mm -> 246.3 x 91 mm
- copper layers 2 -> 4

Commit message: add split sensor board for breakaway
Parts:
- added J2: Conn_01x32_Pin, mine:Conn_1x32_SMD, F.Cu at (166.5, 65.1)
- added J3: Conn_01x32_Pin, mine:Conn_1x32_SMD, F.Cu at (16.5, 51.7)
- added JP24: SolderJumper_2_Open, Jumper:SolderJumper-2_P1.3mm_Open_TrianglePad1.0x1.5mm, F.Cu at (138.7, 67.4)
- added JP25: SolderJumper_2_Open, Jumper:SolderJumper-2_P1.3mm_Open_TrianglePad1.0x1.5mm, F.Cu at (138.7, 70.2)
- added JP26: SolderJumper_2_Open, Jumper:SolderJumper-2_P1.3mm_Open_TrianglePad1.0x1.5mm, F.Cu at (138.7, 73.0)
- added JP5: SolderJumper_2_Open, Jumper:SolderJumper-2_P1.3mm_Open_TrianglePad1.0x1.5mm, F.Cu at (138.7, 58.4)
- added JP6: SolderJumper_2_Open, Jumper:SolderJumper-2_P1.3mm_Open_TrianglePad1.0x1.5mm, F.Cu at (138.7, 61.5)
- added JP7: SolderJumper_2_Open, Jumper:SolderJumper-2_P1.3mm_Open_TrianglePad1.0x1.5mm, F.Cu at (138.8, 64.6)
- interboard connect: renamed from J1
- moved JP23 59.9 mm to (71.4, 85.8)
- moved JPE01 31.5 mm to (23.3, 87.0)
- moved JPE02 31.5 mm to (25.8, 87.0)
- moved JPE03 31.5 mm to (28.3, 87.0)
- moved JPE04 31.5 mm to (30.8, 87.0)
- moved JPE05 31.5 mm to (33.5, 87.0)
- moved JPE06 31.5 mm to (36.0, 87.0)
- moved JPE07 31.5 mm to (38.5, 87.0)
- moved JPE09 31.5 mm to (43.5, 87.0)
- moved JPE10 31.5 mm to (46.0, 87.0)
- moved JPE11 31.5 mm to (48.5, 87.0)
- moved JPE12 31.5 mm to (51.0, 87.0)
- moved JPE14 31.5 mm to (56.0, 87.0)
- moved JPE16 31.5 mm to (61.0, 87.0)
- moved JPE17 31.5 mm to (63.5, 87.0)
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Connections:
- JP10 pad 1: Net-(JP10-A) -> Net-(DG452_0-S_2)
- JP11 pad 1: Net-(JP11-A) -> Net-(DG452_0-D_3)
- JP12 pad 1: Net-(JP12-A) -> Net-(DG452_1-S_1)
- JP13 pad 1: Net-(JP13-A) -> Net-(DG452_1-D_4)
- JP14 pad 1: Net-(JP14-A) -> Net-(DG452_1-S_2)
- JP15 pad 1: Net-(JP15-A) -> Net-(DG452_1-D_3)
- JP16 pad 1: Net-(JP16-A) -> Net-(DG452_2-S_1)
- JP17 pad 1: Net-(JP17-A) -> Net-(DG452_2-D_4)
- JP18 pad 1: Net-(JP18-A) -> Net-(DG452_2-S_2)
- JP19 pad 1: Net-(JP19-A) -> Net-(DG452_2-D_3)
- JP20 pad 1: Net-(JP20-A) -> Net-(DG452_3-S_1)
- JP21 pad 1: Net-(JP21-A) -> Net-(DG452_3-D_4)
- JP22 pad 1: Net-(JP22-A) -> Net-(DG452_3-S_2)
- JP45 pad 1: Net-(JP45-A) -> Net-(DG452_3-D_3)
- JP46 pad 1: Net-(JP46-A) -> Net-(DG45_4-S_1)
- JP47 pad 1: Net-(JP47-A) -> Net-(DG45_4-D_4)
- JP8 pad 1: Net-(JP8-A) -> Net-(DG452_0-S_1)
- JP9 pad 1: Net-(JP9-A) -> Net-(DG452_0-D_4)
- JPE01 pad 1: Net-(JP8-A) -> Net-(DG452_0-S_1)
- JPE02 pad 1: Net-(JP9-A) -> Net-(DG452_0-D_4)
- JPE03 pad 1: Net-(JP10-A) -> Net-(DG452_0-S_2)
- JPE04 pad 1: Net-(JP11-A) -> Net-(DG452_0-D_3)
- JPE05 pad 1: Net-(JP12-A) -> Net-(DG452_1-S_1)
- JPE06 pad 1: Net-(JP13-A) -> Net-(DG452_1-D_4)
- JPE07 pad 1: Net-(JP14-A) -> Net-(DG452_1-S_2)
- JPE08 pad 1: Net-(JP15-A) -> Net-(DG452_1-D_3)
- JPE09 pad 1: Net-(JP16-A) -> Net-(DG452_2-S_1)
- JPE10 pad 1: Net-(JP17-A) -> Net-(DG452_2-D_4)
- JPE11 pad 1: Net-(JP18-A) -> Net-(DG452_2-S_2)
- JPE12 pad 1: Net-(JP19-A) -> Net-(DG452_2-D_3)
- JPE13 pad 1: Net-(JP20-A) -> Net-(DG452_3-S_1)
- JPE14 pad 1: Net-(JP21-A) -> Net-(DG452_3-D_4)
- JPE15 pad 1: Net-(JP22-A) -> Net-(DG452_3-S_2)
- JPE16 pad 1: Net-(JP45-A) -> Net-(DG452_3-D_3)
- JPE17 pad 1: Net-(JP46-A) -> Net-(DG45_4-S_1)
- JPE18 pad 1: Net-(JP47-A) -> Net-(DG45_4-D_4)
- U1 pad 16: Net-(JP8-A) -> Net-(DG452_0-S_1)
- U1 pad 17: Net-(JP9-A) -> Net-(DG452_0-D_4)
- U1 pad 18: Net-(JP10-A) -> Net-(DG452_0-S_2)
- U1 pad 19: Net-(JP11-A) -> Net-(DG452_0-D_3)
- U1 pad 30: Net-(JP15-A) -> Net-(DG452_1-D_3)
- U1 pad 31: Net-(JP14-A) -> Net-(DG452_1-S_2)
- U1 pad 32: Net-(JP13-A) -> Net-(DG452_1-D_4)
- U1 pad 33: Net-(JP12-A) -> Net-(DG452_1-S_1)
- U1 pad 36: Net-(JP47-A) -> Net-(DG45_4-D_4)
- U1 pad 37: Net-(JP46-A) -> Net-(DG45_4-S_1)
- U1 pad 38: Net-(JP45-A) -> Net-(DG452_3-D_3)
- U1 pad 39: Net-(JP22-A) -> Net-(DG452_3-S_2)
- U1 pad 40: Net-(JP21-A) -> Net-(DG452_3-D_4)
- U1 pad 41: Net-(JP20-A) -> Net-(DG452_3-S_1)
- U1 pad 42: Net-(JP19-A) -> Net-(DG452_2-D_3)
- U1 pad 43: Net-(JP18-A) -> Net-(DG452_2-S_2)
- U1 pad 44: Net-(JP17-A) -> Net-(DG452_2-D_4)
- U1 pad 45: Net-(JP16-A) -> Net-(DG452_2-S_1)
- interboard connect pad 02: Net-(JP8-A) -> Net-(DG452_0-S_1)
- interboard connect pad 04: Net-(JP9-A) -> Net-(DG452_0-D_4)
- interboard connect pad 06: Net-(JP10-A) -> Net-(DG452_0-S_2)
- interboard connect pad 08: Net-(JP11-A) -> Net-(DG452_0-D_3)
- interboard connect pad 10: Net-(JP12-A) -> Net-(DG452_1-S_1)
- interboard connect pad 12: Net-(JP13-A) -> Net-(DG452_1-D_4)
- interboard connect pad 14: Net-(JP14-A) -> Net-(DG452_1-S_2)
- interboard connect pad 16: Net-(JP15-A) -> Net-(DG452_1-D_3)
- interboard connect pad 18: Net-(JP16-A) -> Net-(DG452_2-S_1)
- interboard connect pad 20: Net-(JP17-A) -> Net-(DG452_2-D_4)
- interboard connect pad 22: Net-(JP18-A) -> Net-(DG452_2-S_2)
- interboard connect pad 24: Net-(JP19-A) -> Net-(DG452_2-D_3)
- interboard connect pad 26: Net-(JP20-A) -> Net-(DG452_3-S_1)
- interboard connect pad 28: Net-(JP21-A) -> Net-(DG452_3-D_4)
- interboard connect pad 30: Net-(JP22-A) -> Net-(DG452_3-S_2)
- interboard connect pad 32: Net-(JP45-A) -> Net-(DG452_3-D_3)
- interboard connect pad 34: Net-(JP46-A) -> Net-(DG45_4-S_1)
- interboard connect pad 36: Net-(JP47-A) -> Net-(DG45_4-D_4)
Routing:
- net Net-(DG452_0-S_1): track 121.3 -> 353.7 mm, vias 1 -> 4
- net Net-(DG452_0-D_4): track 123.8 -> 348.8 mm, vias 1 -> 4
- net Net-(DG452_0-S_2): track 108.1 -> 331.4 mm, vias 1 -> 4
- net Net-(DG452_0-D_3): track 110.0 -> 326.7 mm, vias 1 -> 4
- net Net-(DG452_1-S_1): track 100.1 -> 300.7 mm, vias 1 -> 4
- net Net-(DG452_1-D_4): track 102.6 -> 295.8 mm, vias 1 -> 4
- net Net-(DG452_1-S_2): track 88.1 -> 279.5 mm, vias 1 -> 4
- net Net-(DG452_1-D_3): track 90.7 -> 276.5 mm, vias 1 -> 4
- net Net-(J2-Pin_9): track 25.3 -> 208.2 mm, vias 0 -> 2
- net Net-(DG452_2-S_1): track 84.1 -> 263.1 mm, vias 1 -> 4
- net Net-(DG452_2-S_2): track 75.3 -> 251.4 mm, vias 1 -> 4
- net Net-(DG452_2-D_4): track 83.2 -> 256.4 mm, vias 1 -> 4
- net Net-(DG45_4-S_1): track 66.4 -> 239.3 mm, vias 1 -> 4
- net Net-(DG452_3-S_1): track 72.4 -> 244.2 mm, vias 1 -> 4
- net Net-(DG452_3-S_2): track 68.7 -> 240.2 mm, vias 1 -> 4
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Other:
- outline, holes or cut-outs redrawn
- board text added: "------ sensor out ---"
- board text added: "--------- sensor out ---------"
- board text added: "0"
- board text added: "0 1 2 3 board select"
- board text added: "1"
- board text added: "18"
- board text added: "2"
- board text added: "3"
- board text added: "3.3v"
- board text added: "< a mid-morning snack"
- board text added: "GND"
- board text added: "I hope you can read this"
- board text added: "I hope you like soldering"
- board text added: "V_IN"
- board text added: "V_IN connect"
- board text added: "^ 1"
- board text added: "^ touch ground to speak to aliens"
- board text added: "board identifier"
- board text added: "key 13 disable"
- board text added: "key 14 disable"
- board text added: "key 15 disable"
- board text added: "key 16 disable"
- board text added: "key 17 disable"
- board text added: "key 18 disable"
- board text added: "lo hi v v"
- board text added: "s1 v"
- board text added: "s18 v"
- board text added: "the ultimate sensor-y experience"
- board text added: "you might not need this"
- board text added: "you probably don't need this"
- board text added: "you should probably keep this"
