File: sampler_split_sensor/sampler_split_sensor.kicad_pcb (KiCad board)
At the start: 4 copper layers, 249 x 115.4 mm, 96 parts, among them J1 TSW-120-20-S-D-LL, J2 Conn_01x32_Pin, J3 Conn_01x32_Pin, J4 Conn_01x32_Pin, J5 Conn_01x32_Pin, U1 Teensy4.1, U10 DRV5055A1xLPGxQ1, U11 DRV5055A1xLPGxQ1, U12 DRV5055A1xLPGxQ1, U13 DRV5055A1xLPGxQ1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

Commit message: Boards v3
Signed-off-by: Sawyer Bergeron <sawyerbergeron@gmail.com>
Other:
- outline, holes or cut-outs redrawn
Changed lines of the file:
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@@
 		(at 90.800001 55 -90)
 		(property "Reference" "J4"
-			(at 0 -0.499999 270)
+			(at 0 -0.499999 -90)
 			(unlocked yes)
 			(layer "F.SilkS")
@@
 		(pts
 			(xy 21 52) (xy 13 44) (xy 13 34) (xy 15.6 31.4) (xy 258.4 31.4) (xy 262 35) (xy 262 40) (xy 250 52)
-			(xy 97 52) (xy 96.8 52.1) (xy 96.8 52.4) (xy 97 52.5) (xy 98 52.5) (xy 100 54.5) (xy 100 63) (xy 103 66)
-			(xy 164 66) (xy 166 68) (xy 169.1 68) (xy 170 68.9) (xy 170 133) (xy 169 134) (xy 163 134) (xy 159 138)
-			(xy 18 138) (xy 14.1 134.1) (xy 14.1 55.5) (xy 17.1 52.5) (xy 22 52.5) (xy 22 52)
+			(xy 97 52) (xy 96.8 52.1) (xy 96.8 52.4) (xy 97 52.5) (xy 98 52.5) (xy 98 52.5) (xy 160.187499 52.5)
+			(xy 160.187499 52.5) (xy 170 52.5) (xy 170 133) (xy 169 134) (xy 163 134) (xy 159 138) (xy 18 138)
+			(xy 14.1 134.1) (xy 14.1 55.5) (xy 17.1 52.5) (xy 22 52.5) (xy 22 52)
 		)
 		(stroke
