File: boards_v3/boards_v3.kicad_pcb (KiCad board)
At the start: 4 copper layers, 155 x 68.1 mm, 50 parts, among them J1 Conn_02x04_Counter_Clockwise, J2 Conn_02x04_Counter_Clockwise, J3 Conn_02x04_Counter_Clockwise, J4 Conn_02x04_Counter_Clockwise, J6 Conn_02x04_Counter_Clockwise, J7 Conn_02x04_Counter_Clockwise, J8 Conn_02x04_Counter_Clockwise, J9 Conn_02x17_Counter_Clockwise, U1 Teensy4.1

Commit message: boards
Signed-off-by: Sawyer Bergeron <sawyerbergeron@gmail.com>
Parts:
- added C1: 0.1uF, Capacitor_SMD:C_1206_3216Metric_Pad1.33x1.80mm_HandSolder, B.Cu at (67.4, 37.5)
- added C10: 0.1uF, Capacitor_SMD:C_1206_3216Metric_Pad1.33x1.80mm_HandSolder, B.Cu at (188.8, 37.5)
- added C11: 0.1uF, Capacitor_SMD:C_1206_3216Metric_Pad1.33x1.80mm_HandSolder, B.Cu at (172.8, 37.5)
- added C12: 0.1uF, Capacitor_SMD:C_1206_3216Metric_Pad1.33x1.80mm_HandSolder, B.Cu at (156.3, 37.5)
- added C13: 0.1uF, Capacitor_SMD:C_1206_3216Metric_Pad1.33x1.80mm_HandSolder, F.Cu at (193.5, 68.7)
- added C14: 0.1uF, Capacitor_SMD:C_1206_3216Metric_Pad1.33x1.80mm_HandSolder, B.Cu at (123.8, 37.5)
- added C15: 0.1uF, Capacitor_SMD:C_1206_3216Metric_Pad1.33x1.80mm_HandSolder, B.Cu at (132.3, 37.6)
- added C16: 0.1uF, Capacitor_SMD:C_1206_3216Metric_Pad1.33x1.80mm_HandSolder, B.Cu at (148.3, 37.5)
- added C17: C_Small, Capacitor_SMD:C_1206_3216Metric_Pad1.33x1.80mm_HandSolder, B.Cu at (140.3, 37.5)
- added C18: 20uF, Capacitor_SMD:C_1812_4532Metric_Pad1.57x3.40mm_HandSolder, B.Cu at (87.1, 64.5)
- added C2: 0.1uF, Capacitor_SMD:C_1206_3216Metric_Pad1.33x1.80mm_HandSolder, B.Cu at (75.5, 37.5)
- added C3: 0.1uF, Capacitor_SMD:C_1206_3216Metric_Pad1.33x1.80mm_HandSolder, B.Cu at (83.5, 37.5)
- added C4: 0.1uF, Capacitor_SMD:C_1206_3216Metric_Pad1.33x1.80mm_HandSolder, B.Cu at (164.8, 37.5)
- added C5: 0.1uF, Capacitor_SMD:C_1206_3216Metric_Pad1.33x1.80mm_HandSolder, B.Cu at (180.5, 37.6)
- added C6: 0.1uF, Capacitor_SMD:C_1206_3216Metric_Pad1.33x1.80mm_HandSolder, B.Cu at (91.4, 37.5)
- added C7: 0.1uF, Capacitor_SMD:C_1206_3216Metric_Pad1.33x1.80mm_HandSolder, B.Cu at (99.7, 37.5)
- added C8: 0.1uF, Capacitor_SMD:C_1206_3216Metric_Pad1.33x1.80mm_HandSolder, B.Cu at (107.9, 37.5)
- added C9: 0.1uF, Capacitor_SMD:C_1206_3216Metric_Pad1.33x1.80mm_HandSolder, B.Cu at (115.9, 37.5)
Routing:
- net GND: track 25.8 -> 217.2 mm, vias 42 -> 57
- net +3.3V: track 562.6 -> 576.0 mm
- net +5V: track 233.5 -> 244.7 mm
- net Net-(J9-Pin_7): track 143.3 -> 146.0 mm
- net Net-(U10-~E): track 206.2 -> 207.7 mm, vias 19 -> 17
- net Net-(J6-Pin_5): track 61.9 -> 63.3 mm, vias 0 -> 1
- net Net-(J6-Pin_4): track 72.5 -> 73.4 mm, vias 0 -> 1
- net Net-(J9-Pin_9): track 153.4 -> 152.7 mm
- net Net-(J9-Pin_2): track 111.9 -> 112.4 mm
- added copper zone on B.Cu, net +3.3V
- added copper zone on In1.Cu, net GND
Other:
- board text added: "(also)"
- board text added: "+3.3V"
- board text added: "+5V"
- board text added: "0....................7 board select"
- board text added: "0........3 comm"
- board text added: "0.1µF"
- board text added: "1 ------------ sensors ------------ 16"
- board text added: "20µF"
- board text added: "A1"
- board text added: "A2"
- board text added: "CMP CHIP"
- board text added: "D1"
- board text added: "D2"
- board text added: "D3"
- board text added: "D4"
- board text added: "D5"
- board text added: "SPST Switch"
- board text added: "board select 1 - 2 - 4 - 8 - 16 - 32 - 64 - 128"

Commit message: iter
Signed-off-by: Sawyer Bergeron <sawyerbergeron@gmail.com>
Connections:
- U1 pad 16: Net-(J9-Pin_6) -> Net-(J9-Pin_1)
- U1 pad 17: Net-(J9-Pin_5) -> Net-(J9-Pin_2)
- U1 pad 18: Net-(J9-Pin_4) -> Net-(J9-Pin_3)
- U1 pad 19: Net-(J9-Pin_3) -> Net-(J9-Pin_4)
- U1 pad 26: Net-(J6-Pin_5) -> Net-(J6-Pin_4)
- U1 pad 27: Net-(J6-Pin_4) -> Net-(J6-Pin_5)
- U1 pad 30: Net-(J8-Pin_2) -> Net-(J8-Pin_1)
- U1 pad 31: Net-(J8-Pin_1) -> Net-(J8-Pin_2)
- U1 pad 32: Net-(J9-Pin_2) -> Net-(J9-Pin_5)
- U1 pad 33: Net-(J9-Pin_1) -> Net-(J9-Pin_6)
- U1 pad 36: Net-(J9-Pin_16) -> Net-(J9-Pin_7)
- U1 pad 37: Net-(J9-Pin_15) -> Net-(J9-Pin_8)
- U1 pad 38: Net-(J9-Pin_14) -> Net-(J9-Pin_9)
- U1 pad 39: Net-(J9-Pin_13) -> Net-(J9-Pin_10)
- U1 pad 40: Net-(J9-Pin_12) -> Net-(J9-Pin_11)
- U1 pad 41: Net-(J9-Pin_11) -> Net-(J9-Pin_12)
- U1 pad 42: Net-(J9-Pin_10) -> Net-(J9-Pin_13)
- U1 pad 43: Net-(J9-Pin_9) -> Net-(J9-Pin_14)
- U1 pad 44: Net-(J9-Pin_8) -> Net-(J9-Pin_15)
- U1 pad 45: Net-(J9-Pin_7) -> Net-(J9-Pin_16)
Routing:
- net Net-(J9-Pin_6): track 171.7 -> 108.3 mm, vias 3 -> 2
- net Net-(J9-Pin_5): track 159.7 -> 106.6 mm, vias 3 -> 2
- net Net-(J9-Pin_9): track 152.7 -> 124.1 mm, vias 3 -> 2
- net Net-(J9-Pin_7): track 146.0 -> 118.3 mm, vias 3 -> 2
- net Net-(J9-Pin_16): track 224.6 -> 197.1 mm, vias 3 -> 2
- net Net-(J9-Pin_4): track 148.0 -> 120.5 mm, vias 3 -> 2
- net Net-(J9-Pin_10): track 158.2 -> 131.0 mm, vias 3 -> 2
- net Net-(J9-Pin_11): track 163.3 -> 137.4 mm, vias 3 -> 2
- net Net-(J9-Pin_8): track 146.1 -> 121.0 mm, vias 3 -> 2
- net Net-(J9-Pin_15): track 205.3 -> 184.1 mm, vias 3 -> 2
- net Net-(J9-Pin_12): track 169.0 -> 148.0 mm, vias 3 -> 2
- net Net-(J9-Pin_14): track 189.8 -> 170.7 mm, vias 3 -> 2
- net Net-(J9-Pin_13): track 176.7 -> 159.5 mm, vias 3 -> 2
- net Net-(J9-Pin_3): track 136.8 -> 121.5 mm, vias 3 -> 2
- net Net-(U10-~E): track 207.7 -> 193.0 mm
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Other:
- outline, holes or cut-outs redrawn
