File: boards_v3/boards_v3.kicad_sch (KiCad schematic)
At the start: 50 parts, among them J1 Conn_02x04_Counter_Clockwise, J2 Conn_02x04_Counter_Clockwise, J3 Conn_02x04_Counter_Clockwise, J4 Conn_02x04_Counter_Clockwise, J6 Conn_02x04_Counter_Clockwise, J7 Conn_02x04_Counter_Clockwise, J8 Conn_02x04_Counter_Clockwise, J9 Conn_02x17_Counter_Clockwise, U1 Teensy4.1

Commit message: boards
Signed-off-by: Sawyer Bergeron <sawyerbergeron@gmail.com>
Parts:
- added C1, C10, C11, C12, C13, C14, C15, C16, C2, C3, C4, C5, C6, C7, C8, C9: 0.1uF, Capacitor_SMD:C_1206_3216Metric_Pad1.33x1.80mm_HandSolder, symbol Device:C_Small
- added C17: C_Small, Capacitor_SMD:C_1206_3216Metric_Pad1.33x1.80mm_HandSolder, symbol Device:C_Small
- added C18: 20uF, Capacitor_SMD:C_1812_4532Metric_Pad1.57x3.40mm_HandSolder, symbol Device:C_Small
Connections:
- net +3.3V: now also C1.1, C10.1, C11.1, C12.1, C13.1, C14.1, C15.1, C16.1, C17.1, C2.1, C3.1, C4.1, C5.1, C6.1, C7.1, C8.1, C9.1
- net +5V: now also C18.1
- net GND: now also C1.2, C10.2, C11.2, C12.2, C13.2, C14.2, C15.2, C16.2, C17.2, C18.2, C2.2, C3.2, C4.2, C5.2, C6.2, C7.2, C8.2, C9.2
Other:
- moved on the sheet: J6

Commit message: iter
Signed-off-by: Sawyer Bergeron <sawyerbergeron@gmail.com>
Connections:
- net at J9.4 (Pin_4), JP4.2 (C), U5.1 (Y): now also U1.19 (27_A13_SCK1); no longer U1.18 (26_A12_MOSI1)
- net at J9.16 (Pin_16), JP16.2 (C), U17.1 (Y): now also U1.45 (23_A9_CRX1_MCLK1); no longer U1.36 (14_A0_TX3_SPDIF_OUT)
- net at J9.7 (Pin_7), JP7.2 (C), U8.1 (Y): now also U1.36 (14_A0_TX3_SPDIF_OUT); no longer U1.45 (23_A9_CRX1_MCLK1)
- net at J9.14 (Pin_14), JP14.2 (C), U15.1 (Y): now also U1.43 (21_A7_RX5_BCLK1); no longer U1.38 (16_A2_RX4_SCL1)
- net at J9.12 (Pin_12), JP12.2 (C), U13.1 (Y): now also U1.41 (19_A5_SCL); no longer U1.40 (18_A4_SDA)
- net at J9.10 (Pin_10), JP10.2 (C), U11.1 (Y): now also U1.39 (17_A3_TX4_SDA1); no longer U1.42 (20_A6_TX5_LRCLK1)
- net at J8.1 (Pin_1): now also U1.30 (38_CS1_IN1); no longer U1.31 (39_MISO1_OUT1A)
- net at J8.2 (Pin_2): now also U1.31 (39_MISO1_OUT1A); no longer U1.30 (38_CS1_IN1)
- net at J9.13 (Pin_13), JP13.2 (C), U14.1 (Y): now also U1.42 (20_A6_TX5_LRCLK1); no longer U1.39 (17_A3_TX4_SDA1)
- net at J9.2 (Pin_2), JP2.2 (C), U3.1 (Y): now also U1.17 (25_A11_RX6_SDA2); no longer U1.32 (40_A16)
- net at J9.15 (Pin_15), JP15.2 (C), U16.1 (Y): now also U1.44 (22_A8_CTX1); no longer U1.37 (15_A1_RX3_SPDIF_IN)
- net at J9.9 (Pin_9), JP9.2 (C), U10.1 (Y): now also U1.38 (16_A2_RX4_SCL1); no longer U1.43 (21_A7_RX5_BCLK1)
- net at J9.6 (Pin_6), JP6.2 (C), U7.1 (Y): now also U1.33 (41_A17); no longer U1.16 (24_A10_TX6_SCL2)
- net at J9.5 (Pin_5), JP5.2 (C), U6.1 (Y): now also U1.32 (40_A16); no longer U1.17 (25_A11_RX6_SDA2)
- net at J9.3 (Pin_3), JP3.2 (C), U4.1 (Y): now also U1.18 (26_A12_MOSI1); no longer U1.19 (27_A13_SCK1)
- net at U1.26 (34_RX8): now also J6.4 (Pin_4); no longer J6.5 (Pin_5)
- net at U1.27 (35_TX8): now also J6.5 (Pin_5); no longer J6.4 (Pin_4)
- net at J9.1 (Pin_1), JP1.2 (C), U2.1 (Y): now also U1.16 (24_A10_TX6_SCL2); no longer U1.33 (41_A17)
- net at J9.11 (Pin_11), JP11.2 (C), U12.1 (Y): now also U1.40 (18_A4_SDA); no longer U1.41 (19_A5_SCL)
- net at J9.8 (Pin_8), JP8.2 (C), U9.1 (Y): now also U1.37 (15_A1_RX3_SPDIF_IN); no longer U1.44 (22_A8_CTX1)
