File: boards_v3/sensor_v3.kicad_pcb (KiCad board)
At the start: 2 copper layers, 48.3 x 15 mm, 5 parts, among them J1 Conn_02x04_Counter_Clockwise, U1 DRV5055A1xLPGxQ1, U2 DRV5055A1xLPGxQ1, U3 DRV5055A1xLPGxQ1, U4 DRV5055A1xLPGxQ1

Commit message: fixes
Signed-off-by: Sawyer Bergeron <sawyerbergeron@gmail.com>
Routing:
- net GND: track 72.6 -> 0.00 mm
- added copper zone on B.Cu, net GND
Other:
- outline, holes or cut-outs redrawn
Changed lines of the file:
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@@
 	(gr_poly
 		(pts
-			(xy 19.3 20.7) (xy 21 19) (xy 66.5 19) (xy 67.6 20.1) (xy 67.6 27.4) (xy 66 29) (xy 32 29) (xy 32 31.9)
-			(xy 29.9 34) (xy 20 34) (xy 19.3 33.3)
+			(xy 19.3 20.7) (xy 21 19) (xy 66.5 19) (xy 67.6 20.1) (xy 67.6 27.4) (xy 66 29) (xy 32 29) (xy 32 32.5)
+			(xy 30.5 34) (xy 20 34) (xy 19.3 33.3)
 		)
 		(stroke
@@
 	)
 	(segment
-		(start 23.6 22.76)
-		(end 25.66 20.7)
-		(width 0.2)
-		(layer "B.Cu")
-		(net 7)
-	)
-	(segment
-		(start 45.7 20.7)
-		(end 61.74 20.7)
-		(width 0.2)
-		(layer "B.Cu")
-		(net 7)
-	)
-	(segment
-		(start 48.34 20.7)
-		(end 50.4 22.76)
-		(width 0.2)
-		(layer "B.Cu")
-		(net 7)
-	)
-	(segment
-		(start 20.9 24.2)
-		(end 19.9 25.2)
-		(width 0.2)
-		(layer "B.Cu")
-		(net 7)
-	)
-	(segment
-		(start 21.7 24.2)
-		(end 20.9 24.2)
-		(width 0.2)
-		(layer "B.Cu")
-		(net 7)
-	)
-	(segment
-		(start 34.5 20.7)
-		(end 37.6 20.7)
-		(width 0.2)
-		(layer "B.Cu")
-		(net 7)
-	)
-	(segment
-		(start 23.14 22.76)
-		(end 21.7 24.2)
-		(width 0.2)
-		(layer "B.Cu")
-		(net 7)
-	)
-	(segment
-		(start 25.66 20.7)
-		(end 34.5 20.7)
-		(width 0.2)
-		(layer "B.Cu")
-		(net 7)
-	)
-	(segment
-		(start 37.6 20.7)
-		(end 45.7 20.7)
-		(width 0.2)
-		(layer "B.Cu")
-		(net 7)
-	)
-	(segment
-		(start 27.1905 33.2065)
-		(end 28.6335 31.7635)
-		(width 0.2)
-		(layer "B.Cu")
-		(net 7)
-	)
-	(segment
-		(start 35 20.7)
-		(end 37 22.7)
-		(width 0.2)
-		(layer "B.Cu")
-		(net 7)
-	)
-	(segment
-		(start 45.7 20.7)
-		(end 48.34 20.7)
-		(width 0.2)
-		(layer "B.Cu")
-		(net 7)
-	)
-	(segment
-		(start 20.415789 33.2065)
-		(end 27.1905 33.2065)
-		(width 0.2)
-		(layer "B.Cu")
-		(net 7)
-	)
-	(segment
-		(start 61.74 20.7)
-		(end 63.8 22.76)
-		(width 0.2)
-		(layer "B.Cu")
-		(net 7)
-	)
-	(segment
-		(start 19.9 25.2)
-		(end 19.9 32.690711)
-		(width 0.2)
-		(layer "B.Cu")
-		(net 7)
-	)
-	(segment
-		(start 23.6 22.76)
-		(end 23.14 22.76)
-		(width 0.2)
-		(layer "B.Cu")
-		(net 7)
-	)
-	(segment
-		(start 19.9 32.690711)
-		(end 20.415789 33.2065)
-		(width 0.2)
-		(layer "B.Cu")
-		(net 7)
-	)
-	(segment
-		(start 37 22.7)
-		(end 37 22.76)
-		(width 0.2)
-		(layer "B.Cu")
-		(net 7)
-	)
-	(segment
-		(start 34.5 20.7)
-		(end 35 20.7)
-		(width 0.2)
-		(layer "B.Cu")
-		(net 7)
-	)
-	(segment
 		(start 26.139999 22.76)
 		(end 26.139999 24.540002)
@@
 		(net 8)
 	)
+	(zone
+		(net 7)
+		(net_name "GND")
+		(layer "B.Cu")
+		(hatch edge 0.5)
+		(connect_pads
+			(clearance 0.5)
+		)
+		(min_thickness 0.25)
+		(filled_areas_thickness no)
+		(fill yes
+			(thermal_gap 0.2)
+			(thermal_bridge_width 0.5)
+		)
+		(polygon
+			(pts
+				(xy 21 19.5) (xy 66.5 19.5) (xy 67 20) (xy 67 27) (xy 65.5 28.5) (xy 32 28.5) (xy 32 32) (xy 30 34)
+				(xy 20.5 34) (xy 19.5 32.5) (xy 19.5 21)
+			)
+		)
+	)
 )
